File: pcb/display_group/display_socket.kicad_sch (KiCad schematic)
At the start: 2 parts, among them J14 L, J15 R

Commit message: cleaned up, reworked and (so far) finalized the display-group board
Parts:
- J17: renamed from J14; footprint Connector_PinSocket_2.54mm:PinSocket_1x09_P2.54mm_Vertical_SMD_Pin1Left -> Connector_PinSocket_2.54mm:PinSocket_1x09_P2.54mm_Vertical_SMD_Pin1Right
- J18: renamed from J15; footprint Connector_PinSocket_2.54mm:PinSocket_1x09_P2.54mm_Vertical_SMD_Pin1Left -> Connector_PinSocket_2.54mm:PinSocket_1x09_P2.54mm_Vertical_SMD_Pin1Right
Changed lines of the file:
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@@
   (symbol (lib_id "Connector:Conn_01x09_Female") (at 147.32 102.87 0) (unit 1)
     (in_bom yes) (on_board yes) (dnp no)
-    (property "Reference" "J14" (at 145.796 87.376 0)
+    (property "Reference" "J17" (at 145.796 87.376 0)
       (effects (font (size 1.27 1.27)) (justify left))
     )
@@
       (effects (font (size 1.27 1.27)) (justify left))
     )
-    (property "Footprint" "Connector_PinSocket_2.54mm:PinSocket_1x09_P2.54mm_Vertical_SMD_Pin1Left" (at 147.32 102.87 0)
+    (property "Footprint" "Connector_PinSocket_2.54mm:PinSocket_1x09_P2.54mm_Vertical_SMD_Pin1Right" (at 147.32 102.87 0)
       (effects (font (size 1.27 1.27)) hide)
     )
@@
   (symbol (lib_id "Connector:Conn_01x09_Female") (at 152.4 102.87 0) (mirror y) (unit 1)
     (in_bom yes) (on_board yes) (dnp no) (fields_autoplaced)
-    (property "Reference" "J15" (at 153.035 87.376 0)
+    (property "Reference" "J18" (at 153.035 87.376 0)
       (effects (font (size 1.27 1.27)))
     )
@@
       (effects (font (size 1.27 1.27)))
     )
-    (property "Footprint" "Connector_PinSocket_2.54mm:PinSocket_1x09_P2.54mm_Vertical_SMD_Pin1Left" (at 152.4 102.87 0)
+    (property "Footprint" "Connector_PinSocket_2.54mm:PinSocket_1x09_P2.54mm_Vertical_SMD_Pin1Right" (at 152.4 102.87 0)
       (effects (font (size 1.27 1.27)) hide)
     )
